File: SP_kicad/SP_kicad.kicad_pcb (KiCad board)
At the start: 2 copper layers, 135 x 203 mm, 15 parts, among them J1 NES-CART, J2 NES-CART-CONN, J3 MIDI, J4 5V_IN, SW1 BUS_PWR, SW2 CMOD_PWR, U1 CMOD-A7, U2 LD1117V33

Commit message: Update level shifter placement
Parts:
- turned U2 to 180 degrees
Routing:
- net +3.3V: track 141.7 -> 129.1 mm
- net +5V: track 210.5 -> 218.7 mm
- net GND: track 519.3 -> 515.9 mm
Changed lines of the file:
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@@
   )
   (footprint "LD1117V33:TO255P1020X450X1968-3" (layer "F.Cu")
-    (at 71.95 55.605)
+    (at 71.95 55.605 180)
     (property "Availability" "In Stock")
     (property "Check_prices" "https://www.snapeda.com/parts/LD1117V33/STMicroelectronics/view-part/?ref=eda")
@@
     (fp_line (start 5.1 2.25) (end -5.1 2.25)
       (stroke (width 0.127) (type solid)) (layer "F.Fab"))
-    (pad "1" thru_hole rect (at -2.55 0.605) (size 1.91 1.91) (drill 1.27) (layers "*.Cu" "*.Mask")
+    (pad "1" thru_hole rect (at -2.55 0.605 180) (size 1.91 1.91) (drill 1.27) (layers "*.Cu" "*.Mask")
       (net 26 "GND") (pinfunction "ADJ/GND") (pintype "passive") (solder_mask_margin 0.102))
-    (pad "2" thru_hole circle (at 0 0.605) (size 1.91 1.91) (drill 1.27) (layers "*.Cu" "*.Mask")
+    (pad "2" thru_hole circle (at 0 0.605 180) (size 1.91 1.91) (drill 1.27) (layers "*.Cu" "*.Mask")
       (net 30 "+3.3V") (pinfunction "VOUT") (pintype "output") (solder_mask_margin 0.102))
-    (pad "3" thru_hole circle (at 2.55 0.605) (size 1.91 1.91) (drill 1.27) (layers "*.Cu" "*.Mask")
+    (pad "3" thru_hole circle (at 2.55 0.605 180) (size 1.91 1.91) (drill 1.27) (layers "*.Cu" "*.Mask")
       (net 1 "+5V") (pinfunction "VIN") (pintype "input") (solder_mask_margin 0.102))
   )
@@
     (effects (font (size 1 1) (thickness 0.15)) (justify left bottom))
   )
-  (segment (start 74.5 49.5) (end 74.5 56.21) (width 0.25) (layer "F.Cu") (net 1))
-  (segment (start 69 44) (end 74.5 49.5) (width 0.25) (layer "F.Cu") (net 1))
-  (segment (start 65.7648 63.7352) (end 69.95 59.55) (width 0.25) (layer "F.Cu") (net 1))
+  (segment (start 69.4 55) (end 60.6648 63.7352) (width 0.25) (layer "F.Cu") (net 1))
+  (segment (start 60.6648 63.7352) (end 50.2648 63.7352) (width 0.25) (layer "F.Cu") (net 1))
   (segment (start 50.2648 63.7352) (end 40 74) (width 0.25) (layer "F.Cu") (net 1))
-  (segment (start 71.16 59.55) (end 74.5 56.21) (width 0.25) (layer "F.Cu") (net 1))
-  (segment (start 65.7648 63.7352) (end 50.2648 63.7352) (width 0.25) (layer "F.Cu") (net 1))
-  (segment (start 69.95 59.55) (end 71.16 59.55) (width 0.25) (layer "F.Cu") (net 1))
   (segment (start 132.695 73.8952) (end 106.225 73.8952) (width 0.25) (layer "B.Cu") (net 1))
-  (segment (start 89.235 56.425) (end 74.715 56.425) (width 0.25) (layer "B.Cu") (net 1))
+  (segment (start 90.66 55) (end 89.235 53.575) (width 0.25) (layer "B.Cu") (net 1))
   (segment (start 41.125 72.875) (end 40 74) (width 0.25) (layer "B.Cu") (net 1))
   (segment (start 90.66 47.7) (end 89 46.04) (width 0.25) (layer "B.Cu") (net 1))
+  (segment (start 87.905 47.135) (end 72.135 47.135) (width 0.25) (layer "B.Cu") (net 1))
   (segment (start 104.96 75.16) (end 103.695 73.8952) (width 0.25) (layer "B.Cu") (net 1))
   (segment (start 106.225 73.8952) (end 104.96 75.16) (width 0.25) (layer "B.Cu") (net 1))
   (segment (start 133.96 75.16) (end 132.695 73.8952) (width 0.25) (layer "B.Cu") (net 1))
-  (segment (start 74.715 56.425) (end 74.5 56.21) (width 0.25) (layer "B.Cu") (net 1))
+  (segment (start 89.235 53.575) (end 70.825 53.575) (width 0.25) (layer "B.Cu") (net 1))
   (segment (start 161.575 73.8952) (end 135.225 73.8952) (width 0.25) (layer "B.Cu") (net 1))
   (segment (start 163 75.32) (end 161.575 73.8952) (width 0.25) (layer "B.Cu") (net 1))
+  (segment (start 70.825 53.575) (end 69.4 55) (width 0.25) (layer "B.Cu") (net 1))
   (segment (start 73.175 72.875) (end 41.125 72.875) (width 0.25) (layer "B.Cu") (net 1))
+  (segment (start 89 46.04) (end 87.905 47.135) (width 0.25) (layer "B.Cu") (net 1))
   (segment (start 90.66 55) (end 90.66 47.7) (width 0.25) (layer "B.Cu") (net 1))
   (segment (start 103.695 73.8952) (end 76.7248 73.8952) (width 0.25) (layer "B.Cu") (net 1))
-  (segment (start 90.66 55) (end 89.235 56.425) (width 0.25) (layer "B.Cu") (net 1))
+  (segment (start 72.135 47.135) (end 69 44) (width 0.25) (layer "B.Cu") (net 1))
   (segment (start 75.46 75.16) (end 73.175 72.875) (width 0.25) (layer "B.Cu") (net 1))
   (segment (start 76.7248 73.8952) (end 75.46 75.16) (width 0.25) (layer "B.Cu") (net 1))
@@
   (segment (start 165.585 65.115) (end 165.585 45.175) (width 0.25) (layer "F.Cu") (net 26))
   (segment (start 79.2648 73.8952) (end 78 75.16) (width 0.25) (layer "F.Cu") (net 26))
-  (segment (start 55.187614 56.21) (end 52.375054 53.39744) (width 0.25) (layer "F.Cu") (net 26))
   (segment (start 106.235 73.8952) (end 79.2648 73.8952) (width 0.25) (layer "F.Cu") (net 26))
   (segment (start 137.925 66.4248) (end 164.275 66.4248) (width 0.25) (layer "F.Cu") (net 26))
@@
   (segment (start 169.725 94.3) (end 169.725 79.505) (width 0.25) (layer "F.Cu") (net 26))
   (segment (start 165.585 45.175) (end 167 43.76) (width 0.25) (layer "F.Cu") (net 26))
-  (segment (start 69 55.81) (end 69.4 56.21) (width 0.25) (layer "F.Cu") (net 26))
-  (segment (start 69.4 56.21) (end 55.187614 56.21) (width 0.25) (layer "F.Cu") (net 26))
+  (segment (start 49.22852 51.82022) (end 63.71978 51.82022) (width 0.25) (layer "F.Cu") (net 26))
   (segment (start 164.275 66.4248) (end 165.54 65.16) (width 0.25) (layer "F.Cu") (net 26))
+  (segment (start 74.5 52.04) (end 69 46.54) (width 0.25) (layer "F.Cu") (net 26))
   (segment (start 137.605 74.0552) (end 164.275 74.0552) (width 0.25) (layer "F.Cu") (net 26))
   (segment (start 169.025 95) (end 169.725 94.3) (width 0.25) (layer "F.Cu") (net 26))
@@
   (segment (start 107.5 65) (end 108.765 66.2648) (width 0.25) (layer "F.Cu") (net 26))
   (segment (start 107.5 75.16) (end 106.235 73.8952) (width 0.25) (layer "F.Cu") (net 26))
+  (segment (start 47.6513 53.39744) (end 49.22852 51.82022) (width 0.25) (layer "F.Cu") (net 26))
   (segment (start 136.5 75.16) (end 135.235 73.8952) (width 0.25) (layer "F.Cu") (net 26))
-  (segment (start 69 46.54) (end 69 55.81) (width 0.25) (layer "F.Cu") (net 26))
   (segment (start 135.235 66.2648) (end 136.5 65) (width 0.25) (layer "F.Cu") (net 26))
   (segment (start 136.5 75.16) (end 137.605 74.0552) (width 0.25) (layer "F.Cu") (net 26))
+  (segment (start 74.5 55) (end 74.5 52.04) (width 0.25) (layer "F.Cu") (net 26))
   (segment (start 106.235 66.2648) (end 107.5 65) (width 0.25) (layer "F.Cu") (net 26))
   (segment (start 79.2648 66.2648) (end 106.235 66.2648) (width 0.25) (layer "F.Cu") (net 26))
+  (segment (start 63.71978 51.82022) (end 69 46.54) (width 0.25) (layer "F.Cu") (net 26))
   (segment (start 136.5 65) (end 137.925 66.4248) (width 0.25) (layer "F.Cu") (net 26))
-  (segment (start 52.375054 53.39744) (end 47.6513 53.39744) (width 0.25) (layer "F.Cu") (net 26))
-  (segment (start 52.3751 53.3974) (end 47.6513 53.3974) (width 0.25) (layer "F.Cu") (net 26))
   (segment (start 152.74 95) (end 168 95) (width 0.25) (layer "F.Cu") (net 26))
   (segment (start 164.275 74.0552) (end 165.54 75.32) (width 0.25) (layer "F.Cu") (net 26))
@@
   (segment (start 165.54 65.16) (end 165.585 65.115) (width 0.25) (layer "F.Cu") (net 26))
   (via (at 168 95) (size 0.8) (drill 0.4) (layers "F.Cu" "B.Cu") (net 26))
-  (segment (start 69.4 56.4) (end 78 65) (width 0.25) (layer "B.Cu") (net 26))
   (segment (start 61 157.063) (end 61 227.025) (width 0.25) (layer "B.Cu") (net 26))
+  (segment (start 78 58.5) (end 74.5 55) (width 0.25) (layer "B.Cu") (net 26))
   (segment (start 168 95) (end 123.063 95) (width 0.25) (layer "B.Cu") (net 26))
-  (segment (start 69.4 56.21) (end 69.4 56.4) (width 0.25) (layer "B.Cu") (net 26))
+  (segment (start 78 65) (end 78 58.5) (width 0.25) (layer "B.Cu") (net 26))
   (segment (start 123.063 95) (end 61 157.063) (width 0.25) (layer "B.Cu") (net 26))
   (segment (start 61 227.025) (end 60.0253 228) (width 0.25) (layer "B.Cu") (net 26))
@@
   (segment (start 132.695 66.2648) (end 112.365 66.2648) (width 0.25) (layer "B.Cu") (net 30))
   (segment (start 163 65.16) (end 161.735 66.4248) (width 0.25) (layer "B.Cu") (net 30))
-  (segment (start 62.67 54.93) (end 52.6 65) (width 0.25) (layer "B.Cu") (net 30))
   (segment (start 104.96 65) (end 106.225 66.2648) (width 0.25) (layer "B.Cu") (net 30))
   (segment (start 135.225 66.2648) (end 139.035 66.2648) (width 0.25) (layer "B.Cu") (net 30))
-  (segment (start 71.95 56.21) (end 70.67 54.93) (width 0.25) (layer "B.Cu") (net 30))
+  (segment (start 75.46 58.51) (end 71.95 55) (width 0.25) (layer "B.Cu") (net 30))
   (segment (start 76.7248 66.2648) (end 80.8352 66.2648) (width 0.25) (layer "B.Cu") (net 30))
   (segment (start 109.835 66.2648) (end 111.1 65) (width 0.25) (layer "B.Cu") (net 30))
@@
   (segment (start 80.8352 66.2648) (end 82.1 65) (width 0.25) (layer "B.Cu") (net 30))
   (segment (start 75.46 65) (end 74.1952 66.2648) (width 0.25) (layer "B.Cu") (net 30))
-  (segment (start 70.67 54.93) (end 62.67 54.93) (width 0.25) (layer "B.Cu") (net 30))
   (segment (start 104.96 65) (end 103.695 66.2648) (width 0.25) (layer "B.Cu") (net 30))
   (segment (start 133.96 65) (end 135.225 66.2648) (width 0.25) (layer "B.Cu") (net 30))
@@
   (segment (start 161.735 66.4248) (end 141.405 66.4248) (width 0.25) (layer "B.Cu") (net 30))
   (segment (start 141.405 66.4248) (end 140.14 65.16) (width 0.25) (layer "B.Cu") (net 30))
+  (segment (start 75.46 65) (end 75.46 58.51) (width 0.25) (layer "B.Cu") (net 30))
   (segment (start 83.3648 66.2648) (end 82.1 65) (width 0.25) (layer "B.Cu") (net 30))
   (segment (start 53.8648 66.2648) (end 52.6 65) (width 0.25) (layer "B.Cu") (net 30))
