File: SP_kicad/SP_kicad.kicad_pcb (KiCad board)
At the start: 2 copper layers, 135 x 203 mm, 15 parts, among them J1 NES-CART, J2 NES-CART-CONN, J3 MIDI, J4 5V_IN, SW1 BUS_PWR, SW2 CMOD_PWR, U1 CMOD-A7, U2 LD1117V33

Commit message: Moved Kicad footprints into project
Connections:
- U1 pad 36: Net-(U1-W5) -> unconnected-(U1-W5-Pad36)
- U1 pad 38: Net-(U1-U4) -> unconnected-(U1-U4-Pad38)
- U1 pad 45: unconnected-(U1-U7-Pad45) -> Net-(U1-U7)
- U1 pad 47: unconnected-(U1-U8-Pad47) -> Net-(U1-U8)
- U6 pad 3: Net-(U1-U4) -> Net-(U1-U7)
- U6 pad 5: Net-(U1-W5) -> Net-(U1-U8)
Routing:
- net Net-(U1-W5): track 82.8 -> 0.00 mm
- net Net-(U1-U4): track 71.7 -> 0.00 mm
- net Net-(U1-U8): track 0.00 -> 52.1 mm
- net Net-(U1-U7): track 0.00 -> 52.1 mm
Changed lines of the file:
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@@
   (net 17 "unconnected-(U1-W3-Pad34)")
   (net 18 "unconnected-(U1-V3-Pad35)")
-  (net 19 "Net-(U1-W5)")
+  (net 19 "unconnected-(U1-W5-Pad36)")
   (net 20 "unconnected-(U1-V4-Pad37)")
-  (net 21 "Net-(U1-U4)")
+  (net 21 "unconnected-(U1-U4-Pad38)")
   (net 22 "unconnected-(U1-G3*-Pad15)")
   (net 23 "unconnected-(U1-V5-Pad39)")
@@
   (net 128 "Net-(U1-W6)")
   (net 129 "Net-(U1-U3)")
-  (net 130 "unconnected-(U1-U7-Pad45)")
+  (net 130 "Net-(U1-U7)")
   (net 131 "Net-(U1-W7)")
-  (net 132 "unconnected-(U1-U8-Pad47)")
+  (net 132 "Net-(U1-U8)")
   (net 133 "Net-(U1-V8)")
   (net 134 "Net-(U6-B4)")
@@
       (net 18 "unconnected-(U1-V3-Pad35)") (pinfunction "V3") (pintype "bidirectional+no_connect"))
     (pad "36" thru_hole oval (at 8.636 27.94 90) (size 1.6 1.6) (drill 0.8) (layers "*.Cu" "*.Mask")
-      (net 19 "Net-(U1-W5)") (pinfunction "W5") (pintype "bidirectional"))
+      (net 19 "unconnected-(U1-W5-Pad36)") (pinfunction "W5") (pintype "bidirectional+no_connect"))
     (pad "37" thru_hole oval (at 8.636 25.4 90) (size 1.6 1.6) (drill 0.8) (layers "*.Cu" "*.Mask")
       (net 20 "unconnected-(U1-V4-Pad37)") (pinfunction "V4") (pintype "bidirectional+no_connect"))
     (pad "38" thru_hole oval (at 8.636 22.86 90) (size 1.6 1.6) (drill 0.8) (layers "*.Cu" "*.Mask")
-      (net 21 "Net-(U1-U4)") (pinfunction "U4") (pintype "bidirectional"))
+      (net 21 "unconnected-(U1-U4-Pad38)") (pinfunction "U4") (pintype "bidirectional+no_connect"))
     (pad "39" thru_hole oval (at 8.636 20.32 90) (size 1.6 1.6) (drill 0.8) (layers "*.Cu" "*.Mask")
       (net 23 "unconnected-(U1-V5-Pad39)") (pinfunction "V5") (pintype "bidirectional+no_connect"))
@@
       (net 129 "Net-(U1-U3)") (pinfunction "U3") (pintype "bidirectional"))
     (pad "45" thru_hole oval (at 8.636 5.08 90) (size 1.6 1.6) (drill 0.8) (layers "*.Cu" "*.Mask")
-      (net 130 "unconnected-(U1-U7-Pad45)") (pinfunction "U7") (pintype "bidirectional+no_connect"))
+      (net 130 "Net-(U1-U7)") (pinfunction "U7") (pintype "bidirectional"))
     (pad "46" thru_hole oval (at 8.636 2.54 90) (size 1.6 1.6) (drill 0.8) (layers "*.Cu" "*.Mask")
       (net 131 "Net-(U1-W7)") (pinfunction "W7") (pintype "bidirectional"))
     (pad "47" thru_hole oval (at 8.636 0 90) (size 1.6 1.6) (drill 0.8) (layers "*.Cu" "*.Mask")
-      (net 132 "unconnected-(U1-U8-Pad47)") (pinfunction "U8") (pintype "bidirectional+no_connect"))
+      (net 132 "Net-(U1-U8)") (pinfunction "U8") (pintype "bidirectional"))
     (pad "48" thru_hole oval (at 8.636 -2.54 90) (size 1.6 1.6) (drill 0.8) (layers "*.Cu" "*.Mask")
       (net 133 "Net-(U1-V8)") (pinfunction "V8") (pintype "bidirectional"))
@@
       (net 30 "+3.3V") (pinfunction "VA") (pintype "power_in") (solder_mask_margin 0.0762))
     (pad "3" thru_hole circle (at -7.62 5.08 90) (size 1.8796 1.8796) (drill 1.016) (layers "*.Cu" "*.Mask")
-      (net 21 "Net-(U1-U4)") (pinfunction "A1") (pintype "bidirectional") (solder_mask_margin 0.0762))
+      (net 130 "Net-(U1-U7)") (pinfunction "A1") (pintype "bidirectional") (solder_mask_margin 0.0762))
     (pad "4" thru_hole circle (at -5.08 5.08 90) (size 1.8796 1.8796) (drill 1.016) (layers "*.Cu" "*.Mask")
       (net 131 "Net-(U1-W7)") (pinfunction "A2") (pintype "bidirectional") (solder_mask_margin 0.0762))
     (pad "5" thru_hole circle (at -2.54 5.08 90) (size 1.8796 1.8796) (drill 1.016) (layers "*.Cu" "*.Mask")
-      (net 19 "Net-(U1-W5)") (pinfunction "A3") (pintype "bidirectional") (solder_mask_margin 0.0762))
+      (net 132 "Net-(U1-U8)") (pinfunction "A3") (pintype "bidirectional") (solder_mask_margin 0.0762))
     (pad "6" thru_hole circle (at 0 5.08 90) (size 1.8796 1.8796) (drill 1.016) (layers "*.Cu" "*.Mask")
       (net 133 "Net-(U1-V8)") (pinfunction "A4") (pintype "bidirectional") (solder_mask_margin 0.0762))
@@
   (segment (start 52.6475 56.1925) (end 52.6475 55.8968) (width 0.25) (layer "F.Cu") (net 8))
   (segment (start 45 63.84) (end 52.6475 56.1925) (width 0.25) (layer "F.Cu") (net 8))
-  (segment (start 67.84 65) (end 71.84 61) (width 0.25) (layer "F.Cu") (net 19))
-  (segment (start 80 61) (end 88 53) (width 0.25) (layer "F.Cu") (net 19))
-  (segment (start 88 53) (end 101.88 53) (width 0.25) (layer "F.Cu") (net 19))
-  (segment (start 110.214999 42.185) (end 109.705 42.694999) (width 0.25) (layer "F.Cu") (net 19))
-  (segment (start 137.485 42.185) (end 110.214999 42.185) (width 0.25) (layer "F.Cu") (net 19))
-  (segment (start 71.84 61) (end 80 61) (width 0.25) (layer "F.Cu") (net 19))
-  (segment (start 137.485 42.185) (end 139.06 43.76) (width 0.25) (layer "F.Cu") (net 19))
-  (segment (start 109.705 45.175) (end 101.88 53) (width 0.25) (layer "F.Cu") (net 19))
-  (segment (start 109.705 42.694999) (end 109.705 45.175) (width 0.25) (layer "F.Cu") (net 19))
-  (segment (start 72.92 65) (end 74.92 63) (width 0.25) (layer "F.Cu") (net 21))
-  (segment (start 86.0036 63) (end 94.0036 55) (width 0.25) (layer "F.Cu") (net 21))
-  (segment (start 115.075 43.294009) (end 115.734009 42.635) (width 0.25) (layer "F.Cu") (net 21))
-  (segment (start 115.734009 42.635) (end 132.855 42.635) (width 0.25) (layer "F.Cu") (net 21))
-  (segment (start 74.92 63) (end 86.0036 63) (width 0.25) (layer "F.Cu") (net 21))
-  (segment (start 94.0036 55) (end 104.96 55) (width 0.25) (layer "F.Cu") (net 21))
-  (segment (start 115.075 44.885) (end 115.075 43.294009) (width 0.25) (layer "F.Cu") (net 21))
-  (segment (start 104.96 55) (end 115.075 44.885) (width 0.25) (layer "F.Cu") (net 21))
-  (segment (start 132.855 42.635) (end 133.98 43.76) (width 0.25) (layer "F.Cu") (net 21))
   (segment (start 108.765 73.8952) (end 107.5 75.16) (width 0.25) (layer "F.Cu") (net 26))
   (segment (start 165.54 75.32) (end 165.54 65.16) (width 0.25) (layer "F.Cu") (net 26))
@@
   (segment (start 106.5 56) (end 118.74 43.76) (width 0.25) (layer "F.Cu") (net 129))
   (segment (start 84.64 65) (end 93.64 56) (width 0.25) (layer "F.Cu") (net 129))
+  (segment (start 104.96 55) (end 116.2 43.76) (width 0.25) (layer "F.Cu") (net 130))
+  (segment (start 72.92 65) (end 74.92 63) (width 0.25) (layer "F.Cu") (net 130))
+  (segment (start 86.0036 63) (end 94.0036 55) (width 0.25) (layer "F.Cu") (net 130))
+  (segment (start 74.92 63) (end 86.0036 63) (width 0.25) (layer "F.Cu") (net 130))
+  (segment (start 94.0036 55) (end 104.96 55) (width 0.25) (layer "F.Cu") (net 130))
   (segment (start 73.38 62) (end 86.3672 62) (width 0.25) (layer "F.Cu") (net 131))
   (segment (start 86.3672 62) (end 94.3672 54) (width 0.25) (layer "F.Cu") (net 131))
@@
   (segment (start 70.38 65) (end 73.38 62) (width 0.25) (layer "F.Cu") (net 131))
   (segment (start 94.3672 54) (end 103.42 54) (width 0.25) (layer "F.Cu") (net 131))
+  (segment (start 67.84 65) (end 71.84 61) (width 0.25) (layer "F.Cu") (net 132))
+  (segment (start 80 61) (end 88 53) (width 0.25) (layer "F.Cu") (net 132))
+  (segment (start 88 53) (end 101.88 53) (width 0.25) (layer "F.Cu") (net 132))
+  (segment (start 71.84 61) (end 80 61) (width 0.25) (layer "F.Cu") (net 132))
+  (segment (start 101.88 53) (end 111.12 43.76) (width 0.25) (layer "F.Cu") (net 132))
   (segment (start 70.3 60) (end 65.3 65) (width 0.25) (layer "F.Cu") (net 133))
   (segment (start 108.58 43.76) (end 100.34 52) (width 0.25) (layer "F.Cu") (net 133))

Commit message: Updated M2 and SYSTEM_CLK placement
Connections:
- U1 pad 36: unconnected-(U1-W5-Pad36) -> Net-(U1-W5)
- U1 pad 38: unconnected-(U1-U4-Pad38) -> Net-(U1-U4)
- U1 pad 45: Net-(U1-U7) -> unconnected-(U1-U7-Pad45)
- U1 pad 47: Net-(U1-U8) -> unconnected-(U1-U8-Pad47)
- U6 pad 3: Net-(U1-U7) -> Net-(U1-U4)
- U6 pad 5: Net-(U1-U8) -> Net-(U1-W5)
Routing:
- net Net-(U1-W5): track 0.00 -> 82.8 mm
- net Net-(U1-U4): track 0.00 -> 71.7 mm
- net Net-(U1-U8): track 52.1 -> 0.00 mm
- net Net-(U1-U7): track 52.1 -> 0.00 mm
Changed lines of the file:
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@@
   (net 17 "unconnected-(U1-W3-Pad34)")
   (net 18 "unconnected-(U1-V3-Pad35)")
-  (net 19 "unconnected-(U1-W5-Pad36)")
+  (net 19 "Net-(U1-W5)")
   (net 20 "unconnected-(U1-V4-Pad37)")
-  (net 21 "unconnected-(U1-U4-Pad38)")
+  (net 21 "Net-(U1-U4)")
   (net 22 "unconnected-(U1-G3*-Pad15)")
   (net 23 "unconnected-(U1-V5-Pad39)")
@@
   (net 128 "Net-(U1-W6)")
   (net 129 "Net-(U1-U3)")
-  (net 130 "Net-(U1-U7)")
+  (net 130 "unconnected-(U1-U7-Pad45)")
   (net 131 "Net-(U1-W7)")
-  (net 132 "Net-(U1-U8)")
+  (net 132 "unconnected-(U1-U8-Pad47)")
   (net 133 "Net-(U1-V8)")
   (net 134 "Net-(U6-B4)")
@@
       (net 18 "unconnected-(U1-V3-Pad35)") (pinfunction "V3") (pintype "bidirectional+no_connect"))
     (pad "36" thru_hole oval (at 8.636 27.94 90) (size 1.6 1.6) (drill 0.8) (layers "*.Cu" "*.Mask")
-      (net 19 "unconnected-(U1-W5-Pad36)") (pinfunction "W5") (pintype "bidirectional+no_connect"))
+      (net 19 "Net-(U1-W5)") (pinfunction "W5") (pintype "bidirectional"))
     (pad "37" thru_hole oval (at 8.636 25.4 90) (size 1.6 1.6) (drill 0.8) (layers "*.Cu" "*.Mask")
       (net 20 "unconnected-(U1-V4-Pad37)") (pinfunction "V4") (pintype "bidirectional+no_connect"))
     (pad "38" thru_hole oval (at 8.636 22.86 90) (size 1.6 1.6) (drill 0.8) (layers "*.Cu" "*.Mask")
-      (net 21 "unconnected-(U1-U4-Pad38)") (pinfunction "U4") (pintype "bidirectional+no_connect"))
+      (net 21 "Net-(U1-U4)") (pinfunction "U4") (pintype "bidirectional"))
     (pad "39" thru_hole oval (at 8.636 20.32 90) (size 1.6 1.6) (drill 0.8) (layers "*.Cu" "*.Mask")
       (net 23 "unconnected-(U1-V5-Pad39)") (pinfunction "V5") (pintype "bidirectional+no_connect"))
@@
       (net 129 "Net-(U1-U3)") (pinfunction "U3") (pintype "bidirectional"))
     (pad "45" thru_hole oval (at 8.636 5.08 90) (size 1.6 1.6) (drill 0.8) (layers "*.Cu" "*.Mask")
-      (net 130 "Net-(U1-U7)") (pinfunction "U7") (pintype "bidirectional"))
+      (net 130 "unconnected-(U1-U7-Pad45)") (pinfunction "U7") (pintype "bidirectional+no_connect"))
     (pad "46" thru_hole oval (at 8.636 2.54 90) (size 1.6 1.6) (drill 0.8) (layers "*.Cu" "*.Mask")
       (net 131 "Net-(U1-W7)") (pinfunction "W7") (pintype "bidirectional"))
     (pad "47" thru_hole oval (at 8.636 0 90) (size 1.6 1.6) (drill 0.8) (layers "*.Cu" "*.Mask")
-      (net 132 "Net-(U1-U8)") (pinfunction "U8") (pintype "bidirectional"))
+      (net 132 "unconnected-(U1-U8-Pad47)") (pinfunction "U8") (pintype "bidirectional+no_connect"))
     (pad "48" thru_hole oval (at 8.636 -2.54 90) (size 1.6 1.6) (drill 0.8) (layers "*.Cu" "*.Mask")
       (net 133 "Net-(U1-V8)") (pinfunction "V8") (pintype "bidirectional"))
@@
       (net 30 "+3.3V") (pinfunction "VA") (pintype "power_in") (solder_mask_margin 0.0762))
     (pad "3" thru_hole circle (at -7.62 5.08 90) (size 1.8796 1.8796) (drill 1.016) (layers "*.Cu" "*.Mask")
-      (net 130 "Net-(U1-U7)") (pinfunction "A1") (pintype "bidirectional") (solder_mask_margin 0.0762))
+      (net 21 "Net-(U1-U4)") (pinfunction "A1") (pintype "bidirectional") (solder_mask_margin 0.0762))
     (pad "4" thru_hole circle (at -5.08 5.08 90) (size 1.8796 1.8796) (drill 1.016) (layers "*.Cu" "*.Mask")
       (net 131 "Net-(U1-W7)") (pinfunction "A2") (pintype "bidirectional") (solder_mask_margin 0.0762))
     (pad "5" thru_hole circle (at -2.54 5.08 90) (size 1.8796 1.8796) (drill 1.016) (layers "*.Cu" "*.Mask")
-      (net 132 "Net-(U1-U8)") (pinfunction "A3") (pintype "bidirectional") (solder_mask_margin 0.0762))
+      (net 19 "Net-(U1-W5)") (pinfunction "A3") (pintype "bidirectional") (solder_mask_margin 0.0762))
     (pad "6" thru_hole circle (at 0 5.08 90) (size 1.8796 1.8796) (drill 1.016) (layers "*.Cu" "*.Mask")
       (net 133 "Net-(U1-V8)") (pinfunction "A4") (pintype "bidirectional") (solder_mask_margin 0.0762))
@@
   (segment (start 52.6475 56.1925) (end 52.6475 55.8968) (width 0.25) (layer "F.Cu") (net 8))
   (segment (start 45 63.84) (end 52.6475 56.1925) (width 0.25) (layer "F.Cu") (net 8))
+  (segment (start 67.84 65) (end 71.84 61) (width 0.25) (layer "F.Cu") (net 19))
+  (segment (start 80 61) (end 88 53) (width 0.25) (layer "F.Cu") (net 19))
+  (segment (start 88 53) (end 101.88 53) (width 0.25) (layer "F.Cu") (net 19))
+  (segment (start 110.214999 42.185) (end 109.705 42.694999) (width 0.25) (layer "F.Cu") (net 19))
+  (segment (start 137.485 42.185) (end 110.214999 42.185) (width 0.25) (layer "F.Cu") (net 19))
+  (segment (start 71.84 61) (end 80 61) (width 0.25) (layer "F.Cu") (net 19))
+  (segment (start 137.485 42.185) (end 139.06 43.76) (width 0.25) (layer "F.Cu") (net 19))
+  (segment (start 109.705 45.175) (end 101.88 53) (width 0.25) (layer "F.Cu") (net 19))
+  (segment (start 109.705 42.694999) (end 109.705 45.175) (width 0.25) (layer "F.Cu") (net 19))
+  (segment (start 72.92 65) (end 74.92 63) (width 0.25) (layer "F.Cu") (net 21))
+  (segment (start 86.0036 63) (end 94.0036 55) (width 0.25) (layer "F.Cu") (net 21))
+  (segment (start 115.075 43.294009) (end 115.734009 42.635) (width 0.25) (layer "F.Cu") (net 21))
+  (segment (start 115.734009 42.635) (end 132.855 42.635) (width 0.25) (layer "F.Cu") (net 21))
+  (segment (start 74.92 63) (end 86.0036 63) (width 0.25) (layer "F.Cu") (net 21))
+  (segment (start 94.0036 55) (end 104.96 55) (width 0.25) (layer "F.Cu") (net 21))
+  (segment (start 115.075 44.885) (end 115.075 43.294009) (width 0.25) (layer "F.Cu") (net 21))
+  (segment (start 104.96 55) (end 115.075 44.885) (width 0.25) (layer "F.Cu") (net 21))
+  (segment (start 132.855 42.635) (end 133.98 43.76) (width 0.25) (layer "F.Cu") (net 21))
   (segment (start 108.765 73.8952) (end 107.5 75.16) (width 0.25) (layer "F.Cu") (net 26))
   (segment (start 165.54 75.32) (end 165.54 65.16) (width 0.25) (layer "F.Cu") (net 26))
@@
   (segment (start 106.5 56) (end 118.74 43.76) (width 0.25) (layer "F.Cu") (net 129))
   (segment (start 84.64 65) (end 93.64 56) (width 0.25) (layer "F.Cu") (net 129))
-  (segment (start 104.96 55) (end 116.2 43.76) (width 0.25) (layer "F.Cu") (net 130))
-  (segment (start 72.92 65) (end 74.92 63) (width 0.25) (layer "F.Cu") (net 130))
-  (segment (start 86.0036 63) (end 94.0036 55) (width 0.25) (layer "F.Cu") (net 130))
-  (segment (start 74.92 63) (end 86.0036 63) (width 0.25) (layer "F.Cu") (net 130))
-  (segment (start 94.0036 55) (end 104.96 55) (width 0.25) (layer "F.Cu") (net 130))
   (segment (start 73.38 62) (end 86.3672 62) (width 0.25) (layer "F.Cu") (net 131))
   (segment (start 86.3672 62) (end 94.3672 54) (width 0.25) (layer "F.Cu") (net 131))
@@
   (segment (start 70.38 65) (end 73.38 62) (width 0.25) (layer "F.Cu") (net 131))
   (segment (start 94.3672 54) (end 103.42 54) (width 0.25) (layer "F.Cu") (net 131))
-  (segment (start 67.84 65) (end 71.84 61) (width 0.25) (layer "F.Cu") (net 132))
-  (segment (start 80 61) (end 88 53) (width 0.25) (layer "F.Cu") (net 132))
-  (segment (start 88 53) (end 101.88 53) (width 0.25) (layer "F.Cu") (net 132))
-  (segment (start 71.84 61) (end 80 61) (width 0.25) (layer "F.Cu") (net 132))
-  (segment (start 101.88 53) (end 111.12 43.76) (width 0.25) (layer "F.Cu") (net 132))
   (segment (start 70.3 60) (end 65.3 65) (width 0.25) (layer "F.Cu") (net 133))
   (segment (start 108.58 43.76) (end 100.34 52) (width 0.25) (layer "F.Cu") (net 133))
